File: bldc_hardware_riscv/bldc_hardware_riscv.kicad_sch (KiCad schematic)
At the start: 40 parts

Commit message: add debug RX/TX, fix CH9141K footprint error, add 12V detection
Parts:
- removed U: (no value), symbol Connector:Screw_Terminal_01x04
- added J: Screw_Terminal_01x03, symbol Connector:Screw_Terminal_01x03
- added J: Screw_Terminal_01x04, symbol Connector:Screw_Terminal_01x04
Connections:
- net 3.3V: now also J.2 (Pin_2)
- net GND: now also J.1 (Pin_1), J.1 (Pin_1)
- net SWCK: now also J.3 (Pin_3)
- net SWIO: now also J.4 (Pin_4)
- net AIN_V12V: now reaches U.24 (PA1/ADC1)
- net BOOT1: now reaches U.1, U.37 (PB2/BOOT1)
- net DEBUG_TX: now reaches U.47 (PB10)
- net DEBUG_TX: now also J.2 (Pin_2)
- net DEBUG_RX: now reaches U.48 (PB11)
- net DEBUG_RX: now also J.3 (Pin_3)
Other:
- sheet Driver ports: added ADC_V12V; removed none
