File: bldc_hardware_riscv/bldc_hardware_riscv.kicad_pcb (KiCad board)
At the start: 4 copper layers, 81 x 60 mm, 143 parts, among them J1 USB_B_Micro Vertical, J2 2.00mm JST 6Pin, J3 2.00mm JST 6Pin, J4 Screw_Terminal_01x04, J5 Screw_Terminal_01x03, Q1 80V/200A, Q2 80V/200A, Q3 80V/200A, Q4 80V/200A, Q5 80V/200A, Q6 80V/200A, Q9 FCX495, SW1 B3U-1000P, SW2 B3U-1000P, U1 CH32V307VCT6, U101 MT9222WT-65BR5, U102 MT9222WT-65BR5, U103 MT9222WT-65BR5, U2 XL1509-3.3 XLSEMI, U3 EG2134 EG Micro, U4 XL7046 XLSEMI, U5 RT9058-50GVL Richtek, U6 RT9058-50GVL Richtek, U7 SN65HVD230, U8 CH9141K, X1 Keystone-7693, X2 Keystone-7693, X3 Keystone-7693, X4 Keystone-7693, X5 Keystone-7693, Y1 8MHz 3225, Y2 32MHz 3225

Commit message: add missed caps
Parts:
- added C22: 0.1uF, Capacitor_SMD:C_0805_2012Metric, F.Cu at (96.7, 113.2)
- added C23: 0.1uF, Capacitor_SMD:C_0805_2012Metric, F.Cu at (94.7, 106.3)
- moved R17 6.50 mm to (98.2, 106.6), turned to 0 degrees
- moved Q9 0.30 mm to (94.1, 109.9)
Routing:
- net Net-(D18-K): track 7.87 -> 3.97 mm
- net /Driver/99V: track 25.7 -> 29.3 mm
- net GND: track 110.8 -> 113.4 mm, vias 86 -> 87
- net /Driver/75V: track 14.5 -> 15.7 mm

Commit message: Update WCH LOGO, fixed gbr clearance issue (around MCU range)
Parts:
- added R18: 2K2, Resistor_SMD:R_0603_1608Metric, F.Cu at (128.7, 88.5)
- added R19: 2K2, Resistor_SMD:R_0603_1608Metric, F.Cu at (131.6, 90.4)
- added R20: 2K2, Resistor_SMD:R_0603_1608Metric, F.Cu at (133.1, 89.3)
- moved C22 0.30 mm to (96.7, 113.5)
Routing:
- net /3.3V: track 135.3 -> 138.3 mm, vias 13 -> 14
- net /HALL3: track 17.6 -> 20.2 mm
- net /ADC_EXT: track 38.8 -> 39.3 mm
Other:
- board text removed: "Nanjing Qinheng"
- board text removed: "Say hello to"
- board text removed: "UBCO Bikes"
